Commit message: Update robot_1.xacro

File: robot_1.xacro (robot description, xacro)
@@ -38,5 +38,5 @@
         <parent link="world"/>
         <child link="base_link"/>
-        <origin xyz="0 0 0" rpy="0 0 0"/> <!-- Restored 0.1 m gap as per earlier request -->
+        <origin xyz="0 0 0" rpy="0 0 0"/>
     </joint>
     <link name="base_link">
@@ -46,7 +46,5 @@
                 <cylinder radius="${base_radius}" length="${base_length}"/>
             </geometry>
-            <material name="base_material">
-                <color rgba="0 0 0 1"/> <!-- Fully opaque -->
-            </material>
+            <material name="black"/>
         </visual>
         <collision>
@@ -56,5 +54,5 @@
             </geometry>
         </collision>
-        <xacro:cylinder_inertial mass="1" radius="${base_radius}" length="${base_length}" o_xyz="0 0 ${base_length/2}" o_rpy="0 0 0"/>
+        <xacro:cylinder_inertial mass="2" radius="${base_radius}" length="${base_length}" o_xyz="0 0 ${base_length/2}" o_rpy="0 0 0"/>
     </link>
     <!-- *****LINK 1***** -->
@@ -65,7 +63,5 @@
                 <cylinder radius="${link_1_radius}" length="${link_1_length}"/>
             </geometry>
-            <material name="link_1_material">
-                <color rgba="1 0 0 0.5"/> <!-- Red with 50% transparency -->
-            </material>
+            <material name="red"/>
         </visual>
         <collision>
@@ -82,6 +78,6 @@
         <origin xyz="0 0 ${base_length}" rpy="0 0 0"/>
         <axis xyz="0 0 1"/>
-        <limit lower="${-pi/2}" upper="${pi/2}" velocity="1" effort="100"/>
         <dynamics damping="0.7"/>
+        <limit effort="10" lower="${-pi/2}" upper="${pi/2}" velocity="1"/>
     </joint>
     <!-- *****LINK 2p***** -->
@@ -89,16 +85,14 @@
         <visual>
             <geometry>
-                <sphere radius="0.09"/>
+                <sphere radius="${link_1_radius}"/>
             </geometry>
-            <material name="link_2p_material">
-                <color rgba="1 0.5 0 0.5"/> <!-- Orange with 50% transparency -->
-            </material>
+            <material name="orange"/>
         </visual>
         <collision>
             <geometry>
-                <sphere radius="0.09"/>
+                <sphere radius="${link_1_radius}"/>
             </geometry>
         </collision>
-        <xacro:sphere_inertial mass="0.1" radius="0.09" o_xyz="0 0 0" o_rpy="0 0 0"/>
+        <xacro:sphere_inertial mass="0.1" radius="${link_1_radius}" o_xyz="0 0 0" o_rpy="0 0 0"/>
     </link>
     <joint name="1_to_2p" type="fixed">
@@ -110,19 +104,17 @@
     <link name="link_2">
         <visual>
-            <origin xyz="0 0 ${link_2_length/2}" rpy="0 0 0"/>
+            <origin xyz="${link_2_length/2} 0 0" rpy="0 ${pi/2} 0"/>
             <geometry>
                 <cylinder radius="${link_2_radius}" length="${link_2_length}"/>
             </geometry>
-            <material name="link_2_material">
-                <color rgba="1 0.5 0 0.5"/> <!-- Orange with 50% transparency -->
-            </material>
+            <material name="orange"/>
         </visual>
         <collision>
-            <origin xyz="0 0 ${link_2_length/2}" rpy="0 0 0"/>
+            <origin xyz="${link_2_length/2} 0 0" rpy="0 ${pi/2} 0"/>
             <geometry>
                 <cylinder radius="${link_2_radius}" length="${link_2_length}"/>
             </geometry>
         </collision>
-        <xacro:cylinder_inertial mass="1" radius="${link_2_radius}" length="${link_2_length}" o_xyz="0 0 ${link_2_length/2}" o_rpy="0 0 0"/>
+        <xacro:cylinder_inertial mass="0.5" radius="${link_2_radius}" length="${link_2_length}" o_xyz="${link_2_length/2} 0 0" o_rpy="0 ${pi/2} 0"/>
     </link>
     <joint name="1_to_2" type="revolute">
@@ -130,6 +122,6 @@
         <child link="link_2"/>
         <origin xyz="0 0 ${link_1_length}" rpy="0 0 0"/>
-        <axis xyz="0 1 0"/>
-        <limit lower="-0.52" upper="${pi/2}" velocity="1" effort="100"/>
+        <axis xyz="0 1 0"/> <!-- Corrected to rotate around y for horizontal motion -->
+        <limit effort="10" lower="${-0.52}" upper="${pi/2}" velocity="1"/>
         <dynamics damping="0.7"/>
     </joint>
@@ -138,72 +130,66 @@
         <visual>
             <geometry>
-                <sphere radius="0.06"/>
+                <sphere radius="${link_2_radius}"/>
             </geometry>
-            <material name="link_3p_material">
-                <color rgba="0 1 0 0.5"/>
-            </material>
+            <material name="green"/>
         </visual>
         <collision>
             <geometry>
-                <sphere radius="0.06"/>
+                <sphere radius="${link_2_radius}"/>
             </geometry>
         </collision>
-        <xacro:sphere_inertial mass="0.1" radius="0.06" o_xyz="0 0 0" o_rpy="0 0 0"/>
+        <xacro:sphere_inertial mass="0.1" radius="${link_2_radius}" o_xyz="0 0 0" o_rpy="0 0 0"/>
     </link>
     <joint name="2_to_3p" type="fixed">
         <parent link="link_2"/>
         <child link="link_3p"/>
-        <origin xyz="0 0 ${link_2_length}" rpy="0 0 0"/>
+        <origin xyz="${link_2_length} 0 0" rpy="0 0 0"/>
     </joint>
     <!-- *****LINK 3***** -->
     <link name="link_3">
         <visual>
-            <origin xyz="0 0 ${link_3_length/2}" rpy="0 0 0"/>
+            <origin xyz="${link_3_length/2} 0 0" rpy="0 ${pi/2} 0"/>
             <geometry>
                 <cylinder radius="${link_3_radius}" length="${link_3_length}"/>
             </geometry>
-            <material name="link_3_material">
-                <color rgba="0 1 0 0.5"/> <!-- Green with 50% transparency -->
-            </material>
+            <material name="green"/>
         </visual>
         <collision>
-            <origin xyz="0 0 ${link_3_length/2}" rpy="0 0 0"/>
+            <origin xyz="${link_3_length/2} 0 0" rpy="0 ${pi/2} 0"/>
             <geometry>
                 <cylinder radius="${link_3_radius}" length="${link_3_length}"/>
             </geometry>
         </collision>
-        <xacro:cylinder_inertial mass="1" radius="${link_3_radius}" length="${link_3_length}" o_xyz="0 0 ${link_3_length/2}" o_rpy="0 0 0"/>
+        <xacro:cylinder_inertial mass="0.5" radius="${link_3_radius}" length="${link_3_length}" o_xyz="${link_3_length/2} 0 0" o_rpy="0 ${pi/2} 0"/>
     </link>
     <joint name="2_to_3" type="revolute">
         <parent link="link_2"/>
         <child link="link_3"/>
-        <origin xyz="0 0 ${link_2_length}" rpy="0 0 0"/>
-        <axis xyz="1 0 0"/>
-        <limit lower="${-pi/2}" upper="0" velocity="1" effort="100"/>
+        <origin xyz="${link_2_length} 0 0" rpy="0 0 0"/>
+        <axis xyz="1 0 0"/> <!-- Rotate around x for next segment -->
         <dynamics damping="0.7"/>
+        <limit effort="10" lower="${-pi/2}" upper="${0}" velocity="1"/>
     </joint>
     <!-- *****LINK 4***** -->
     <link name="link_4">
         <visual>
-            <origin xyz="0 0 ${link_4_length/2}" rpy="0 0 0"/>
+            <origin xyz="${link_4_length/2} 0 0" rpy="0 ${pi/2} 0"/>
             <geometry>
                 <cylinder radius="${link_4_radius}" length="${link_4_length}"/>
             </geometry>
-            <material name="link_4_material">
-                <color rgba="0 0 1 0.5"/> <!-- Blue with 50% transparency -->
-            </material>
+            <material name="blue"/>
         </visual>
         <collision>
-            <origin xyz="0 0 ${link_4_length/2}" rpy="0 0 0"/>
+            <origin xyz="${link_4_length/2} 0 0" rpy="0 ${pi/2} 0"/>
             <geometry>
                 <cylinder radius="${link_4_radius}" length="${link_4_length}"/>
             </geometry>
         </collision>
-        <xacro:cylinder_inertial mass="1" radius="${link_4_radius}" length="${link_4_length}" o_xyz="0 0 ${link_4_length/2}" o_rpy="0 0 0"/>
+        <xacro:cylinder_inertial mass="0.1" radius="${link_4_radius}" length="${link_4_length}" o_xyz="${link_4_length/2} 0 0" o_rpy="0 ${pi/2} 0"/>
     </link>
     <joint name="3_to_4" type="fixed">
         <parent link="link_3"/>
         <child link="link_4"/>
-        <origin xyz="0 0 ${link_3_length}" rpy="0 0 0"/>
+        <origin xyz="${link_3_length} 0 0" rpy="0 0 0"/>
     </joint>
 </robot>

Commit message: Update robot_1.xacro

File: robot_1.xacro (robot description, xacro)
@@ -21,5 +21,5 @@
             <mass value="${mass}"/>
             <inertia ixx="${mass*(3*radius*radius+length*length)/12}" ixy="0.0" ixz="0.0"
-                     iyy="${mass*(3*radius*radius+length*length)/12}" iyz="0.0" izz="${mass*radius*radius/2}"/>
+            iyy="${mass*(3*radius*radius+length*length)/12}" iyz="0.0" izz="${mass*radius*radius/2}"/>
         </inertial>
     </xacro:macro>
@@ -32,11 +32,10 @@
         </inertial>
     </xacro:macro>
-    <!-- *****World link (no visual geometry)***** -->
+    <!-- *****Base link***** -->
     <link name="world"/>
-    <!-- *****Base link***** -->
     <joint name="world_to_base" type="fixed">
         <parent link="world"/>
         <child link="base_link"/>
-        <origin xyz="0 0 0" rpy="0 0 0"/>
+        <origin xyz="0 0 ${+base_length/2+link_1_length}"/>
     </joint>
     <link name="base_link">
@@ -46,6 +45,9 @@
                 <cylinder radius="${base_radius}" length="${base_length}"/>
             </geometry>
-            <material name="black"/>
-        </visual>
+            <material name="base_material">
+                <color rgba="0 0 0 1"/>
+            </material>
+        </visual>
+        <xacro:cylinder_inertial mass="1" radius="${base_radius}" length="${base_length}" o_xyz="0 0 ${base_length/2}" o_rpy="0 0 0"/>
         <collision>
             <origin xyz="0 0 ${base_length/2}" rpy="0 0 0"/>
@@ -54,5 +56,4 @@
             </geometry>
         </collision>
-        <xacro:cylinder_inertial mass="2" radius="${base_radius}" length="${base_length}" o_xyz="0 0 ${base_length/2}" o_rpy="0 0 0"/>
     </link>
     <!-- *****LINK 1***** -->
@@ -63,6 +64,9 @@
                 <cylinder radius="${link_1_radius}" length="${link_1_length}"/>
             </geometry>
-            <material name="red"/>
-        </visual>
+            <material name="link_1_material">
+                <color rgba="1 0 0 0.5"/>
+            </material>
+        </visual>
+        <xacro:cylinder_inertial mass="1" radius="${link_1_radius}" length="${link_1_length}" o_xyz="0 0 ${link_1_length/2}" o_rpy="0 0 0"/>
         <collision>
             <origin xyz="0 0 ${link_1_length/2}" rpy="0 0 0"/>
@@ -71,13 +75,12 @@
             </geometry>
         </collision>
-        <xacro:cylinder_inertial mass="1" radius="${link_1_radius}" length="${link_1_length}" o_xyz="0 0 ${link_1_length/2}" o_rpy="0 0 0"/>
     </link>
     <joint name="base_to_1" type="revolute">
+        <origin xyz="0 0 0"/>
         <parent link="base_link"/>
         <child link="link_1"/>
-        <origin xyz="0 0 ${base_length}" rpy="0 0 0"/>
         <axis xyz="0 0 1"/>
         <dynamics damping="0.7"/>
-        <limit effort="10" lower="${-pi/2}" upper="${pi/2}" velocity="1"/>
+        <limit effort="100" lower="${-pi/2}" upper="${pi/2}" velocity="1"/>
     </joint>
     <!-- *****LINK 2p***** -->
@@ -85,43 +88,47 @@
         <visual>
             <geometry>
-                <sphere radius="${link_1_radius}"/>
-            </geometry>
-            <material name="orange"/>
-        </visual>
-        <collision>
-            <geometry>
-                <sphere radius="${link_1_radius}"/>
-            </geometry>
-        </collision>
-        <xacro:sphere_inertial mass="0.1" radius="${link_1_radius}" o_xyz="0 0 0" o_rpy="0 0 0"/>
+                <sphere radius="0.09"/>
+            </geometry>
+            <material name="link_2p_material">
+                <color rgba="1 0.5 0 0.5"/>
+            </material>
+        </visual>
+        <xacro:sphere_inertial mass="0.1" radius="0.09" o_xyz="0 0 0" o_rpy="0 0 0"/>
+        <collision>
+            <geometry>
+                <sphere radius="0.09"/>
+            </geometry>
+        </collision>
     </link>
     <joint name="1_to_2p" type="fixed">
         <parent link="link_1"/>
         <child link="link_2p"/>
-        <origin xyz="0 0 ${link_1_length}" rpy="0 0 0"/>
+        <origin xyz="0 0 0"/>
     </joint>
     <!-- *****LINK 2***** -->
     <link name="link_2">
         <visual>
-            <origin xyz="${link_2_length/2} 0 0" rpy="0 ${pi/2} 0"/>
+            <origin xyz="0 0 ${link_2_length/2}" rpy="0 0 0"/>
             <geometry>
                 <cylinder radius="${link_2_radius}" length="${link_2_length}"/>
             </geometry>
-            <material name="orange"/>
-        </visual>
-        <collision>
-            <origin xyz="${link_2_length/2} 0 0" rpy="0 ${pi/2} 0"/>
+            <material name="link_2_material">
+                <color rgba="1 0.5 0 0.5"/>
+            </material>
+        </visual>
+        <xacro:cylinder_inertial mass="1" radius="${link_2_radius}" length="${link_2_length}" o_xyz="0 0 ${link_2_length/2}" o_rpy="0 0 0"/>
+        <collision>
+            <origin xyz="0 0 ${link_2_length/2}" rpy="0 0 0"/>
             <geometry>
                 <cylinder radius="${link_2_radius}" length="${link_2_length}"/>
             </geometry>
         </collision>
-        <xacro:cylinder_inertial mass="0.5" radius="${link_2_radius}" length="${link_2_length}" o_xyz="${link_2_length/2} 0 0" o_rpy="0 ${pi/2} 0"/>
     </link>
     <joint name="1_to_2" type="revolute">
+        <origin xyz="0 0 0" rpy="${pi/2} 0 0"/>
         <parent link="link_1"/>
         <child link="link_2"/>
-        <origin xyz="0 0 ${link_1_length}" rpy="0 0 0"/>
-        <axis xyz="0 1 0"/> <!-- Corrected to rotate around y for horizontal motion -->
-        <limit effort="10" lower="${-0.52}" upper="${pi/2}" velocity="1"/>
+        <axis xyz="0 0 1"/>
+        <limit effort="100" lower="${-0.52}" upper="${pi/2}" velocity="1"/>
         <dynamics damping="0.7"/>
     </joint>
@@ -130,66 +137,73 @@
         <visual>
             <geometry>
-                <sphere radius="${link_2_radius}"/>
-            </geometry>
-            <material name="green"/>
-        </visual>
-        <collision>
-            <geometry>
-                <sphere radius="${link_2_radius}"/>
-            </geometry>
-        </collision>
-        <xacro:sphere_inertial mass="0.1" radius="${link_2_radius}" o_xyz="0 0 0" o_rpy="0 0 0"/>
+                <sphere radius="0.06"/>
+            </geometry>
+            <material name="link_3p_material">
+                <color rgba="0 1 0 0.5"/>
+            </material>
+        </visual>
+        <xacro:sphere_inertial mass="0.1" radius="0.06" o_xyz="0 0 0" o_rpy="0 0 0"/>
+        <collision>
+            <geometry>
+                <sphere radius="0.06"/>
+            </geometry>
+        </collision>
     </link>
     <joint name="2_to_3p" type="fixed">
+        <origin xyz="${link_2_length} 0 0" rpy="0 0 0"/>
         <parent link="link_2"/>
         <child link="link_3p"/>
-        <origin xyz="${link_2_length} 0 0" rpy="0 0 0"/>
     </joint>
     <!-- *****LINK 3***** -->
     <link name="link_3">
         <visual>
-            <origin xyz="${link_3_length/2} 0 0" rpy="0 ${pi/2} 0"/>
+            <origin xyz="0 0 ${link_3_length/2}" rpy="0 0 0"/>
             <geometry>
                 <cylinder radius="${link_3_radius}" length="${link_3_length}"/>
             </geometry>
-            <material name="green"/>
-        </visual>
-        <collision>
-            <origin xyz="${link_3_length/2} 0 0" rpy="0 ${pi/2} 0"/>
+            <material name="link_3_material">
+                <color rgba="0 1 0 0.5"/>
+            </material>
+        </visual>
+        <xacro:cylinder_inertial mass="1" radius="${link_3_radius}" length="${link_3_length}" o_xyz="0 0 ${link_3_length/2}" o_rpy="0 0 0"/>
+        <collision>
+            <origin xyz="0 0 ${link_3_length/2}" rpy="0 0 0"/>
             <geometry>
                 <cylinder radius="${link_3_radius}" length="${link_3_length}"/>
             </geometry>
         </collision>
-        <xacro:cylinder_inertial mass="0.5" radius="${link_3_radius}" length="${link_3_length}" o_xyz="${link_3_length/2} 0 0" o_rpy="0 ${pi/2} 0"/>
     </link>
     <joint name="2_to_3" type="revolute">
+        <origin xyz="${link_2_length} 0 0"/>
         <parent link="link_2"/>
         <child link="link_3"/>
-        <origin xyz="${link_2_length} 0 0" rpy="0 0 0"/>
-        <axis xyz="1 0 0"/> <!-- Rotate around x for next segment -->
+        <axis xyz="0 0 1"/>
         <dynamics damping="0.7"/>
-        <limit effort="10" lower="${-pi/2}" upper="${0}" velocity="1"/>
+        <limit effort="100" lower="${-pi/2}" upper="${0}" velocity="1"/>
     </joint>
     <!-- *****LINK 4***** -->
     <link name="link_4">
         <visual>
-            <origin xyz="${link_4_length/2} 0 0" rpy="0 ${pi/2} 0"/>
+            <origin xyz="0 0 ${link_4_length/2}" rpy="0 0 0"/>
             <geometry>
                 <cylinder radius="${link_4_radius}" length="${link_4_length}"/>
             </geometry>
-            <material name="blue"/>
-        </visual>
-        <collision>
-            <origin xyz="${link_4_length/2} 0 0" rpy="0 ${pi/2} 0"/>
+            <material name="link_4_material">
+                <color rgba="0 0 1 0.5"/>
+            </material>
+        </visual>
+        <xacro:cylinder_inertial mass="1" radius="${link_4_radius}" length="${link_4_length}" o_xyz="0 0 ${link_4_length/2}" o_rpy="0 0 0"/>
+        <collision>
+            <origin xyz="0 0 ${link_4_length/2}" rpy="0 0 0"/>
             <geometry>
                 <cylinder radius="${link_4_radius}" length="${link_4_length}"/>
             </geometry>
         </collision>
-        <xacro:cylinder_inertial mass="0.1" radius="${link_4_radius}" length="${link_4_length}" o_xyz="${link_4_length/2} 0 0" o_rpy="0 ${pi/2} 0"/>
     </link>
     <joint name="3_to_4" type="fixed">
+        <origin xyz="${link_4_length+link_3_length} 0 0"/>
         <parent link="link_3"/>
         <child link="link_4"/>
-        <origin xyz="${link_3_length} 0 0" rpy="0 0 0"/>
+        <axis xyz="0 0 1"/>
     </joint>
 </robot>

Commit message: Update robot_1.xacro

File: robot_1.xacro (robot description, xacro)
@@ -37,5 +37,5 @@
         <parent link="world"/>
         <child link="base_link"/>
-        <origin xyz="0 0 ${+base_length/2+link_1_length}"/>
+        <origin xyz="0 0 0" rpy="0 0 0"/>
     </joint>
     <link name="base_link">
@@ -77,5 +77,5 @@
     </link>
     <joint name="base_to_1" type="revolute">
-        <origin xyz="0 0 0"/>
+        <origin xyz="0 0 ${base_length}" rpy="0 0 0"/>
         <parent link="base_link"/>
         <child link="link_1"/>
@@ -104,5 +104,5 @@
         <parent link="link_1"/>
         <child link="link_2p"/>
-        <origin xyz="0 0 0"/>
+        <origin xyz="0 0 ${link_1_length}" rpy="0 0 0"/>
     </joint>
     <!-- *****LINK 2***** -->
@@ -126,8 +126,8 @@
     </link>
     <joint name="1_to_2" type="revolute">
-        <origin xyz="0 0 0" rpy="${pi/2} 0 0"/>
+        <origin xyz="0 0 ${link_1_length}" rpy="0 0 0"/>
         <parent link="link_1"/>
         <child link="link_2"/>
-        <axis xyz="0 0 1"/>
+        <axis xyz="0 1 0"/>
         <limit effort="100" lower="${-0.52}" upper="${pi/2}" velocity="1"/>
         <dynamics damping="0.7"/>
@@ -151,5 +151,5 @@
     </link>
     <joint name="2_to_3p" type="fixed">
-        <origin xyz="${link_2_length} 0 0" rpy="0 0 0"/>
+        <origin xyz="0 0 ${link_2_length}" rpy="0 0 0"/>
         <parent link="link_2"/>
         <child link="link_3p"/>
@@ -175,8 +175,8 @@
     </link>
     <joint name="2_to_3" type="revolute">
-        <origin xyz="${link_2_length} 0 0"/>
+        <origin xyz="0 0 ${link_2_length}" rpy="0 0 0"/>
         <parent link="link_2"/>
         <child link="link_3"/>
-        <axis xyz="0 0 1"/>
+        <axis xyz="1 0 0"/>
         <dynamics damping="0.7"/>
         <limit effort="100" lower="${-pi/2}" upper="${0}" velocity="1"/>
@@ -202,8 +202,7 @@
     </link>
     <joint name="3_to_4" type="fixed">
-        <origin xyz="${link_4_length+link_3_length} 0 0"/>
+        <origin xyz="0 0 ${link_3_length}" rpy="0 0 0"/>
         <parent link="link_3"/>
         <child link="link_4"/>
-        <axis xyz="0 0 1"/>
     </joint>
 </robot>
