Commit message: Update robot_1.xacro

File: robot_1.xacro (robot description, xacro)
@@ -21,188 +21,148 @@
             <mass value="${mass}"/>
             <inertia ixx="${mass*(3*radius*radius+length*length)/12}" ixy="0.0" ixz="0.0"
-            iyy="${mass*(3*radius*radius+length*length)/12}" iyz="0.0" izz="${mass*radius*radius/2}"/>
+                     iyy="${mass*(3*radius*radius+length*length)/12}" iyz="0.0" izz="${mass*radius*radius/2}"/>
         </inertial>
     </xacro:macro>
-    <xacro:macro name="sphere_inertial" params="mass radius o_xyz o_rpy">
-        <inertial>
-            <origin xyz="${o_xyz}" rpy="${o_rpy}"/>
-            <mass value="${mass}"/>
-            <inertia ixx="${2*mass*radius*radius/5}" ixy="0.0" ixz="0.0"
-                     iyy="${2*mass*radius*radius/5}" iyz="0.0" izz="${2*mass*radius*radius/5}"/>
-        </inertial>
-    </xacro:macro>
+    <!-- *****World link***** -->
+    <link name="world"/>
     <!-- *****Base link***** -->
-    <link name="world"/>
     <joint name="world_to_base" type="fixed">
         <parent link="world"/>
         <child link="base_link"/>
-        <origin xyz="0 0 0" rpy="0 0 0"/>
+        <origin xyz="0 0 ${base_length/2 + link_1_length}" rpy="0 0 0"/>
     </joint>
     <link name="base_link">
         <visual>
-            <origin xyz="0 0 ${base_length/2}" rpy="0 0 0"/>
+            <origin xyz="0 0 ${-base_length/2 - link_1_length}" rpy="0 0 0"/>
             <geometry>
                 <cylinder radius="${base_radius}" length="${base_length}"/>
             </geometry>
-            <material name="base_material">
-                <color rgba="0 0 0 1"/>
-            </material>
+            <material name="black"/>
         </visual>
-        <xacro:cylinder_inertial mass="1" radius="${base_radius}" length="${base_length}" o_xyz="0 0 ${base_length/2}" o_rpy="0 0 0"/>
         <collision>
-            <origin xyz="0 0 ${base_length/2}" rpy="0 0 0"/>
+            <origin xyz="0 0 ${-base_length/2 - link_1_length}" rpy="0 0 0"/>
             <geometry>
                 <cylinder radius="${base_radius}" length="${base_length}"/>
             </geometry>
         </collision>
+        <xacro:cylinder_inertial mass="2" radius="${base_radius}" length="${base_length}" o_xyz="0 0 ${-base_length/2 - link_1_length}" o_rpy="0 0 0"/>
     </link>
     <!-- *****LINK 1***** -->
     <link name="link_1">
         <visual>
-            <origin xyz="0 0 ${link_1_length/2}" rpy="0 0 0"/>
+            <origin xyz="0 0 ${-link_1_length/2}" rpy="0 0 0"/>
             <geometry>
                 <cylinder radius="${link_1_radius}" length="${link_1_length}"/>
             </geometry>
-            <material name="link_1_material">
-                <color rgba="1 0 0 0.5"/>
-            </material>
+            <material name="red"/>
         </visual>
-        <xacro:cylinder_inertial mass="1" radius="${link_1_radius}" length="${link_1_length}" o_xyz="0 0 ${link_1_length/2}" o_rpy="0 0 0"/>
         <collision>
-            <origin xyz="0 0 ${link_1_length/2}" rpy="0 0 0"/>
+            <origin xyz="0 0 ${-link_1_length/2}" rpy="0 0 0"/>
             <geometry>
                 <cylinder radius="${link_1_radius}" length="${link_1_length}"/>
             </geometry>
         </collision>
+        <xacro:cylinder_inertial mass="1" radius="${link_1_radius}" length="${link_1_length}" o_xyz="0 0 ${-link_1_length/2}" o_rpy="0 0 0"/>
     </link>
     <joint name="base_to_1" type="revolute">
-        <origin xyz="0 0 ${base_length}" rpy="0 0 0"/>
         <parent link="base_link"/>
         <child link="link_1"/>
+        <origin xyz="0 0 0" rpy="0 0 0"/>
         <axis xyz="0 0 1"/>
+        <limit lower="${-pi/2}" upper="${pi/2}" velocity="1" effort="10"/>
         <dynamics damping="0.7"/>
-        <limit effort="100" lower="${-pi/2}" upper="${pi/2}" velocity="1"/>
     </joint>
-    <!-- *****LINK 2p***** -->
+    <!-- *****LINK 2p (sphérique)***** -->
     <link name="link_2p">
         <visual>
             <geometry>
-                <sphere radius="0.09"/>
+                <sphere radius="${link_1_radius}"/>
             </geometry>
-            <material name="link_2p_material">
-                <color rgba="1 0.5 0 0.5"/>
-            </material>
+            <material name="orange"/>
         </visual>
-        <xacro:sphere_inertial mass="0.1" radius="0.09" o_xyz="0 0 0" o_rpy="0 0 0"/>
-        <collision>
-            <geometry>
-                <sphere radius="0.09"/>
-            </geometry>
-        </collision>
     </link>
     <joint name="1_to_2p" type="fixed">
         <parent link="link_1"/>
         <child link="link_2p"/>
-        <origin xyz="0 0 ${link_1_length}" rpy="0 0 0"/>
+        <origin xyz="0 0 0" rpy="0 0 0"/>
     </joint>
     <!-- *****LINK 2***** -->
     <link name="link_2">
         <visual>
-            <origin xyz="0 0 ${link_2_length/2}" rpy="0 0 0"/>
+            <origin xyz="${link_2_length/2} 0 0" rpy="0 ${pi/2} 0"/>
             <geometry>
                 <cylinder radius="${link_2_radius}" length="${link_2_length}"/>
             </geometry>
-            <material name="link_2_material">
-                <color rgba="1 0.5 0 0.5"/>
-            </material>
+            <material name="orange"/>
         </visual>
-        <xacro:cylinder_inertial mass="1" radius="${link_2_radius}" length="${link_2_length}" o_xyz="0 0 ${link_2_length/2}" o_rpy="0 0 0"/>
         <collision>
-            <origin xyz="0 0 ${link_2_length/2}" rpy="0 0 0"/>
+            <origin xyz="${link_2_length/2} 0 0" rpy="0 ${pi/2} 0"/>
             <geometry>
                 <cylinder radius="${link_2_radius}" length="${link_2_length}"/>
             </geometry>
         </collision>
+        <xacro:cylinder_inertial mass="0.5" radius="${link_2_radius}" length="${link_2_length}" o_xyz="${link_2_length/2} 0 0" o_rpy="0 ${pi/2} 0"/>
     </link>
     <joint name="1_to_2" type="revolute">
-        <origin xyz="0 0 ${link_1_length}" rpy="0 0 0"/>
         <parent link="link_1"/>
         <child link="link_2"/>
-        <axis xyz="0 1 0"/>
-        <limit effort="100" lower="${-0.52}" upper="${pi/2}" velocity="1"/>
+        <origin xyz="0 0 0" rpy="${pi/2} 0 0"/>
+        <axis xyz="0 0 1"/>
+        <limit lower="-0.52" upper="${pi/2}" velocity="1" effort="10"/>
         <dynamics damping="0.7"/>
     </joint>
-    <!-- *****LINK 3p***** -->
+    <!-- *****LINK 3p (sphérique)***** -->
     <link name="link_3p">
         <visual>
             <geometry>
-                <sphere radius="0.06"/>
+                <sphere radius="${link_2_radius}"/>
             </geometry>
-            <material name="link_3p_material">
-                <color rgba="0 1 0 0.5"/>
-            </material>
+            <material name="green"/>
         </visual>
-        <xacro:sphere_inertial mass="0.1" radius="0.06" o_xyz="0 0 0" o_rpy="0 0 0"/>
-        <collision>
-            <geometry>
-                <sphere radius="0.06"/>
-            </geometry>
-        </collision>
     </link>
     <joint name="2_to_3p" type="fixed">
-        <origin xyz="0 0 ${link_2_length}" rpy="0 0 0"/>
         <parent link="link_2"/>
         <child link="link_3p"/>
+        <origin xyz="${link_2_length} 0 0" rpy="0 0 0"/>
     </joint>
     <!-- *****LINK 3***** -->
     <link name="link_3">
         <visual>
-            <origin xyz="0 0 ${link_3_length/2}" rpy="0 0 0"/>
+            <origin xyz="${link_3_length/2} 0 0" rpy="0 ${pi/2} 0"/>
             <geometry>
                 <cylinder radius="${link_3_radius}" length="${link_3_length}"/>
             </geometry>
-            <material name="link_3_material">
-                <color rgba="0 1 0 0.5"/>
-            </material>
+            <material name="green"/>
         </visual>
-        <xacro:cylinder_inertial mass="1" radius="${link_3_radius}" length="${link_3_length}" o_xyz="0 0 ${link_3_length/2}" o_rpy="0 0 0"/>
         <collision>
-            <origin xyz="0 0 ${link_3_length/2}" rpy="0 0 0"/>
+            <origin xyz="${link_3_length/2} 0 0" rpy="0 ${pi/2} 0"/>
             <geometry>
                 <cylinder radius="${link_3_radius}" length="${link_3_length}"/>
             </geometry>
         </collision>
+        <xacro:cylinder_inertial mass="0.5" radius="${link_3_radius}" length="${link_3_length}" o_xyz="${link_3_length/2} 0 0" o_rpy="0 ${pi/2} 0"/>
     </link>
     <joint name="2_to_3" type="revolute">
-        <origin xyz="0 0 ${link_2_length}" rpy="0 0 0"/>
         <parent link="link_2"/>
         <child link="link_3"/>
-        <axis xyz="1 0 0"/>
+        <origin xyz="${link_2_length} 0 0" rpy="0 0 0"/>
+        <axis xyz="0 0 1"/>
+        <limit lower="${-pi/2}" upper="0" velocity="1" effort="10"/>
         <dynamics damping="0.7"/>
-        <limit effort="100" lower="${-pi/2}" upper="${0}" velocity="1"/>
     </joint>
     <!-- *****LINK 4***** -->
     <link name="link_4">
         <visual>
-            <origin xyz="0 0 ${link_4_length/2}" rpy="0 0 0"/>
+            <origin xyz="${-link_4_length/2} 0 0" rpy="0 ${pi/2} 0"/>
             <geometry>
                 <cylinder radius="${link_4_radius}" length="${link_4_length}"/>
             </geometry>
-            <material name="link_4_material">
-                <color rgba="0 0 1 0.5"/>
-            </material>
+            <material name="blue"/>
         </visual>
-        <xacro:cylinder_inertial mass="1" radius="${link_4_radius}" length="${link_4_length}" o_xyz="0 0 ${link_4_length/2}" o_rpy="0 0 0"/>
-        <collision>
-            <origin xyz="0 0 ${link_4_length/2}" rpy="0 0 0"/>
-            <geometry>
-                <cylinder radius="${link_4_radius}" length="${link_4_length}"/>
-            </geometry>
-        </collision>
     </link>
     <joint name="3_to_4" type="fixed">
-        <origin xyz="0 0 ${link_3_length}" rpy="0 0 0"/>
         <parent link="link_3"/>
         <child link="link_4"/>
+        <origin xyz="${link_3_length + link_4_length} 0 0" rpy="0 0 0"/>
     </joint>
 </robot>

Commit message: Update robot_1.xacro

File: robot_1.xacro (robot description, xacro)
@@ -30,9 +30,9 @@
         <parent link="world"/>
         <child link="base_link"/>
-        <origin xyz="0 0 ${base_length/2 + link_1_length}" rpy="0 0 0"/>
+        <origin xyz="0 0 ${base_length/2}" rpy="0 0 0"/>
     </joint>
     <link name="base_link">
         <visual>
-            <origin xyz="0 0 ${-base_length/2 - link_1_length}" rpy="0 0 0"/>
+            <origin xyz="0 0 ${base_length/2}" rpy="0 0 0"/>
             <geometry>
                 <cylinder radius="${base_radius}" length="${base_length}"/>
@@ -41,15 +41,15 @@
         </visual>
         <collision>
-            <origin xyz="0 0 ${-base_length/2 - link_1_length}" rpy="0 0 0"/>
+            <origin xyz="0 0 ${base_length/2}" rpy="0 0 0"/>
             <geometry>
                 <cylinder radius="${base_radius}" length="${base_length}"/>
             </geometry>
         </collision>
-        <xacro:cylinder_inertial mass="2" radius="${base_radius}" length="${base_length}" o_xyz="0 0 ${-base_length/2 - link_1_length}" o_rpy="0 0 0"/>
+        <xacro:cylinder_inertial mass="2" radius="${base_radius}" length="${base_length}" o_xyz="0 0 ${base_length/2}" o_rpy="0 0 0"/>
     </link>
     <!-- *****LINK 1***** -->
     <link name="link_1">
         <visual>
-            <origin xyz="0 0 ${-link_1_length/2}" rpy="0 0 0"/>
+            <origin xyz="0 0 ${link_1_length/2}" rpy="0 0 0"/>
             <geometry>
                 <cylinder radius="${link_1_radius}" length="${link_1_length}"/>
@@ -58,15 +58,15 @@
         </visual>
         <collision>
-            <origin xyz="0 0 ${-link_1_length/2}" rpy="0 0 0"/>
+            <origin xyz="0 0 ${link_1_length/2}" rpy="0 0 0"/>
             <geometry>
                 <cylinder radius="${link_1_radius}" length="${link_1_length}"/>
             </geometry>
         </collision>
-        <xacro:cylinder_inertial mass="1" radius="${link_1_radius}" length="${link_1_length}" o_xyz="0 0 ${-link_1_length/2}" o_rpy="0 0 0"/>
+        <xacro:cylinder_inertial mass="1" radius="${link_1_radius}" length="${link_1_length}" o_xyz="0 0 ${link_1_length/2}" o_rpy="0 0 0"/>
     </link>
     <joint name="base_to_1" type="revolute">
         <parent link="base_link"/>
         <child link="link_1"/>
-        <origin xyz="0 0 0" rpy="0 0 0"/>
+        <origin xyz="0 0 ${base_length}" rpy="0 0 0"/>
         <axis xyz="0 0 1"/>
         <limit lower="${-pi/2}" upper="${pi/2}" velocity="1" effort="10"/>
@@ -85,5 +85,5 @@
         <parent link="link_1"/>
         <child link="link_2p"/>
-        <origin xyz="0 0 0" rpy="0 0 0"/>
+        <origin xyz="0 0 ${link_1_length}" rpy="0 0 0"/>
     </joint>
     <!-- *****LINK 2***** -->
@@ -107,5 +107,5 @@
         <parent link="link_1"/>
         <child link="link_2"/>
-        <origin xyz="0 0 0" rpy="${pi/2} 0 0"/>
+        <origin xyz="0 0 ${link_1_length}" rpy="${pi/2} 0 0"/>
         <axis xyz="0 0 1"/>
         <limit lower="-0.52" upper="${pi/2}" velocity="1" effort="10"/>

Commit message: Update robot_1.xacro

File: robot_1.xacro (robot description, xacro)
@@ -21,57 +21,60 @@
             <mass value="${mass}"/>
             <inertia ixx="${mass*(3*radius*radius+length*length)/12}" ixy="0.0" ixz="0.0"
-                     iyy="${mass*(3*radius*radius+length*length)/12}" iyz="0.0" izz="${mass*radius*radius/2}"/>
+            iyy="${mass*(3*radius*radius+length*length)/12}" iyz="0.0" izz="${mass*radius*radius/2}"/>
         </inertial>
     </xacro:macro>
-    <!-- *****World link***** -->
+    <!-- *****Base link***** -->
     <link name="world"/>
-    <!-- *****Base link***** -->
     <joint name="world_to_base" type="fixed">
         <parent link="world"/>
         <child link="base_link"/>
-        <origin xyz="0 0 ${base_length/2}" rpy="0 0 0"/>
+        <origin xyz="0 0 ${+base_length/2+link_1_length}"/>
     </joint>
     <link name="base_link">
         <visual>
-            <origin xyz="0 0 ${base_length/2}" rpy="0 0 0"/>
+            <origin xyz="0 0 ${-base_length/2-link_1_length}"/>
             <geometry>
                 <cylinder radius="${base_radius}" length="${base_length}"/>
             </geometry>
-            <material name="black"/>
+            <material name="base_material">
+                <color rgba="0 0 0 0.5"/> <!-- Black with 50% transparency -->
+            </material>
         </visual>
+        <xacro:cylinder_inertial mass="2" radius="${base_radius}" length="${base_length}" o_xyz="0 0 ${base_length/2+link_1_length}" o_rpy="0 0 0"/>
         <collision>
-            <origin xyz="0 0 ${base_length/2}" rpy="0 0 0"/>
+            <origin xyz="0 0 ${-base_length/2-link_1_length}"/>
             <geometry>
                 <cylinder radius="${base_radius}" length="${base_length}"/>
             </geometry>
         </collision>
-        <xacro:cylinder_inertial mass="2" radius="${base_radius}" length="${base_length}" o_xyz="0 0 ${base_length/2}" o_rpy="0 0 0"/>
     </link>
     <!-- *****LINK 1***** -->
     <link name="link_1">
         <visual>
-            <origin xyz="0 0 ${link_1_length/2}" rpy="0 0 0"/>
+            <origin xyz="0 0 ${-link_1_length/2}"/>
             <geometry>
                 <cylinder radius="${link_1_radius}" length="${link_1_length}"/>
             </geometry>
-            <material name="red"/>
+            <material name="link_1_material">
+                <color rgba="1 0 0 0.5"/> <!-- Red with 50% transparency -->
+            </material>
         </visual>
+        <xacro:cylinder_inertial mass="1" radius="${link_1_radius}" length="${link_1_length}" o_xyz="0 0 ${-link_1_length/2}" o_rpy="0 0 0"/>
         <collision>
-            <origin xyz="0 0 ${link_1_length/2}" rpy="0 0 0"/>
+            <origin xyz="0 0 ${-link_1_length/2}"/>
             <geometry>
                 <cylinder radius="${link_1_radius}" length="${link_1_length}"/>
             </geometry>
         </collision>
-        <xacro:cylinder_inertial mass="1" radius="${link_1_radius}" length="${link_1_length}" o_xyz="0 0 ${link_1_length/2}" o_rpy="0 0 0"/>
     </link>
     <joint name="base_to_1" type="revolute">
+        <origin xyz="0 0 0"/>
         <parent link="base_link"/>
         <child link="link_1"/>
-        <origin xyz="0 0 ${base_length}" rpy="0 0 0"/>
         <axis xyz="0 0 1"/>
-        <limit lower="${-pi/2}" upper="${pi/2}" velocity="1" effort="10"/>
         <dynamics damping="0.7"/>
+        <limit effort="10" lower="${-pi/2}" upper="${pi/2}" velocity="1"/>
     </joint>
-    <!-- *****LINK 2p (sphérique)***** -->
+    <!-- *****LINK 2***** -->
     <link name="link_2p">
         <visual>
@@ -79,5 +82,7 @@
                 <sphere radius="${link_1_radius}"/>
             </geometry>
-            <material name="orange"/>
+            <material name="link_2p_material">
+                <color rgba="1 0.5 0 0.5"/> <!-- Orange with 50% transparency -->
+            </material>
         </visual>
     </link>
@@ -85,7 +90,5 @@
         <parent link="link_1"/>
         <child link="link_2p"/>
-        <origin xyz="0 0 ${link_1_length}" rpy="0 0 0"/>
     </joint>
-    <!-- *****LINK 2***** -->
     <link name="link_2">
         <visual>
@@ -94,6 +97,9 @@
                 <cylinder radius="${link_2_radius}" length="${link_2_length}"/>
             </geometry>
-            <material name="orange"/>
+            <material name="link_2_material">
+                <color rgba="1 0.5 0 0.5"/> <!-- Orange with 50% transparency -->
+            </material>
         </visual>
+        <xacro:cylinder_inertial mass="0.5" radius="${link_2_radius}" length="${link_2_length}" o_xyz="${link_2_length/2} 0 0" o_rpy="0 ${pi/2} 0"/>
         <collision>
             <origin xyz="${link_2_length/2} 0 0" rpy="0 ${pi/2} 0"/>
@@ -102,15 +108,14 @@
             </geometry>
         </collision>
-        <xacro:cylinder_inertial mass="0.5" radius="${link_2_radius}" length="${link_2_length}" o_xyz="${link_2_length/2} 0 0" o_rpy="0 ${pi/2} 0"/>
-    </link>
+    </xacro:macro>
     <joint name="1_to_2" type="revolute">
+        <origin xyz="0 0 0" rpy="${pi/2} 0 0"/>
         <parent link="link_1"/>
         <child link="link_2"/>
-        <origin xyz="0 0 ${link_1_length}" rpy="${pi/2} 0 0"/>
         <axis xyz="0 0 1"/>
-        <limit lower="-0.52" upper="${pi/2}" velocity="1" effort="10"/>
+        <limit effort="10" lower="${-0.52}" upper="${pi/2}" velocity="1"/>
         <dynamics damping="0.7"/>
     </joint>
-    <!-- *****LINK 3p (sphérique)***** -->
+    <!-- *****LINK 3***** -->
     <link name="link_3p">
         <visual>
@@ -118,13 +123,14 @@
                 <sphere radius="${link_2_radius}"/>
             </geometry>
-            <material name="green"/>
+            <material name="link_3p_material">
+                <color rgba="0 1 0 0.5"/> <!-- Green with 50% transparency -->
+            </material>
         </visual>
     </link>
-    <joint name="2_to_3p" type="fixed">
+    <joint name="1_to_3p" type="fixed">
+        <origin xyz="${link_2_length} 0 0" rpy="0 0 0"/>
         <parent link="link_2"/>
         <child link="link_3p"/>
-        <origin xyz="${link_2_length} 0 0" rpy="0 0 0"/>
     </joint>
-    <!-- *****LINK 3***** -->
     <link name="link_3">
         <visual>
@@ -133,21 +139,17 @@
                 <cylinder radius="${link_3_radius}" length="${link_3_length}"/>
             </geometry>
-            <material name="green"/>
+            <material name="link_3_material">
+                <color rgba="0 1 0 0.5"/> <!-- Green with 50% transparency -->
+            </material>
         </visual>
-        <collision>
-            <origin xyz="${link_3_length/2} 0 0" rpy="0 ${pi/2} 0"/>
-            <geometry>
-                <cylinder radius="${link_3_radius}" length="${link_3_length}"/>
-            </geometry>
-        </collision>
         <xacro:cylinder_inertial mass="0.5" radius="${link_3_radius}" length="${link_3_length}" o_xyz="${link_3_length/2} 0 0" o_rpy="0 ${pi/2} 0"/>
     </link>
     <joint name="2_to_3" type="revolute">
+        <origin xyz="${link_2_length} 0 0"/>
         <parent link="link_2"/>
         <child link="link_3"/>
-        <origin xyz="${link_2_length} 0 0" rpy="0 0 0"/>
         <axis xyz="0 0 1"/>
-        <limit lower="${-pi/2}" upper="0" velocity="1" effort="10"/>
         <dynamics damping="0.7"/>
+        <limit effort="10" lower="${-pi/2}" upper="${0}" velocity="1"/>
     </joint>
     <!-- *****LINK 4***** -->
@@ -158,11 +160,15 @@
                 <cylinder radius="${link_4_radius}" length="${link_4_length}"/>
             </geometry>
-            <material name="blue"/>
+            <material name="link_4_material">
+                <color rgba="0 0 1 0.5"/> <!-- Blue with 50% transparency -->
+            </material>
         </visual>
     </link>
     <joint name="3_to_4" type="fixed">
+        <origin xyz="${link_4_length+link_3_length} 0 0"/>
         <parent link="link_3"/>
         <child link="link_4"/>
-        <origin xyz="${link_3_length + link_4_length} 0 0" rpy="0 0 0"/>
+        <axis xyz="0 0 1"/>
+        <dynamics damping="0.7"/>
     </joint>
 </robot>

Commit message: Update robot_1.xacro

File: robot_1.xacro (robot description, xacro)
@@ -108,5 +108,5 @@
             </geometry>
         </collision>
-    </xacro:macro>
+    </link>
     <joint name="1_to_2" type="revolute">
         <origin xyz="0 0 0" rpy="${pi/2} 0 0"/>
