Commit message: Update robot_1.xacro

File: robot_1.xacro (robot description, xacro)
@@ -1,4 +1,4 @@
 <?xml version='1.0'?>
-<robot name="robot_ipsa" xmlns:xacro="http://www.ros.org/wiki/xacro">
+<robot name="robot_ipsa" xmlns:xacrowriter.comhttp://www.ros.org/wiki/xacro">
     <xacro:include filename="$(find in426_desc)/xacro/material.xacro"/>
     <xacro:include filename="$(find in426_desc)/xacro/Robot_1/robot_1_ros2_control.xacro"/>
@@ -21,5 +21,13 @@
             <mass value="${mass}"/>
             <inertia ixx="${mass*(3*radius*radius+length*length)/12}" ixy="0.0" ixz="0.0"
-            iyy="${mass*(3*radius*radius+length*length)/12}" iyz="0.0" izz="${mass*radius*radius/2}"/>
+                     iyy="${mass*(3*radius*radius+length*length)/12}" iyz="0.0" izz="${mass*radius*radius/2}"/>
+        </inertial>
+    </xacro:macro>
+    <xacro:macro name="sphere_inertial" params="mass radius o_xyz o_rpy">
+        <inertial>
+            <origin xyz="${o_xyz}" rpy="${o_rpy}"/>
+            <mass value="${mass}"/>
+            <inertia ixx="${2*mass*radius*radius/5}" ixy="0.0" ixz="0.0"
+                     iyy="${2*mass*radius*radius/5}" iyz="0.0" izz="${2*mass*radius*radius/5}"/>
         </inertial>
     </xacro:macro>
@@ -29,9 +37,9 @@
         <parent link="world"/>
         <child link="base_link"/>
-        <origin xyz="0 0 ${+base_length/2+link_1_length}"/>
+        <origin xyz="0 0 ${base_length/2}"/>
     </joint>
     <link name="base_link">
         <visual>
-            <origin xyz="0 0 ${-base_length/2-link_1_length}"/>
+            <origin xyz="0 0 ${base_length/2}" rpy="0 0 0"/>
             <geometry>
                 <cylinder radius="${base_radius}" length="${base_length}"/>
@@ -41,7 +49,7 @@
             </material>
         </visual>
-        <xacro:cylinder_inertial mass="2" radius="${base_radius}" length="${base_length}" o_xyz="0 0 ${base_length/2+link_1_length}" o_rpy="0 0 0"/>
-        <collision>
-            <origin xyz="0 0 ${-base_length/2-link_1_length}"/>
+        <xacro:cylinder_inertial mass="1" radius="${base_radius}" length="${base_length}" o_xyz="0 0 ${base_length/2}" o_rpy="0 0 0"/>
+        <collision>
+            <origin xyz="0 0 ${base_length/2}" rpy="0 0 0"/>
             <geometry>
                 <cylinder radius="${base_radius}" length="${base_length}"/>
@@ -52,5 +60,5 @@
     <link name="link_1">
         <visual>
-            <origin xyz="0 0 ${-link_1_length/2}"/>
+            <origin xyz="0 0 ${link_1_length/2}" rpy="0 0 0"/>
             <geometry>
                 <cylinder radius="${link_1_radius}" length="${link_1_length}"/>
@@ -60,7 +68,7 @@
             </material>
         </visual>
-        <xacro:cylinder_inertial mass="1" radius="${link_1_radius}" length="${link_1_length}" o_xyz="0 0 ${-link_1_length/2}" o_rpy="0 0 0"/>
-        <collision>
-            <origin xyz="0 0 ${-link_1_length/2}"/>
+        <xacro:cylinder_inertial mass="1" radius="${link_1_radius}" length="${link_1_length}" o_xyz="0 0 ${link_1_length/2}" o_rpy="0 0 0"/>
+        <collision>
+            <origin xyz="0 0 ${link_1_length/2}" rpy="0 0 0"/>
             <geometry>
                 <cylinder radius="${link_1_radius}" length="${link_1_length}"/>
@@ -69,10 +77,10 @@
     </link>
     <joint name="base_to_1" type="revolute">
-        <origin xyz="0 0 0"/>
+        <origin xyz="0 0 ${base_length}" rpy="0 0 0"/>
         <parent link="base_link"/>
         <child link="link_1"/>
         <axis xyz="0 0 1"/>
         <dynamics damping="0.7"/>
-        <limit effort="10" lower="${-pi/2}" upper="${pi/2}" velocity="1"/>
+        <limit effort="100" lower="${-pi/2}" upper="${pi/2}" velocity="1"/>
     </joint>
     <!-- *****LINK 2***** -->
@@ -86,6 +94,14 @@
             </material>
         </visual>
+        <xacro:sphere_inertial mass="0.1" radius="${link_1_radius}" o_xyz="0 0 0" o_rpy="0 0 0"/>
+        <collision>
+            <origin xyz="0 0 0" rpy="0 0 0"/>
+            <geometry>
+                <sphere radius="${link_1_radius}"/>
+            </geometry>
+        </collision>
     </link>
     <joint name="1_to_2p" type="fixed">
+        <origin xyz="0 0 ${link_1_length}" rpy="0 0 0"/>
         <parent link="link_1"/>
         <child link="link_2p"/>
@@ -93,5 +109,5 @@
     <link name="link_2">
         <visual>
-            <origin xyz="${link_2_length/2} 0 0" rpy="0 ${pi/2} 0"/>
+            <origin xyz="0 0 ${link_2_length/2}" rpy="0 0 0"/>
             <geometry>
                 <cylinder radius="${link_2_radius}" length="${link_2_length}"/>
@@ -101,7 +117,7 @@
             </material>
         </visual>
-        <xacro:cylinder_inertial mass="0.5" radius="${link_2_radius}" length="${link_2_length}" o_xyz="${link_2_length/2} 0 0" o_rpy="0 ${pi/2} 0"/>
-        <collision>
-            <origin xyz="${link_2_length/2} 0 0" rpy="0 ${pi/2} 0"/>
+        <xacro:cylinder_inertial mass="1" radius="${link_2_radius}" length="${link_2_length}" o_xyz="0 0 ${link_2_length/2}" o_rpy="0 0 0"/>
+        <collision>
+            <origin xyz="0 0 ${link_2_length/2}" rpy="0 0 0"/>
             <geometry>
                 <cylinder radius="${link_2_radius}" length="${link_2_length}"/>
@@ -110,10 +126,10 @@
     </link>
     <joint name="1_to_2" type="revolute">
-        <origin xyz="0 0 0" rpy="${pi/2} 0 0"/>
+        <origin xyz="0 0 ${link_1_length}" rpy="0 0 0"/>
         <parent link="link_1"/>
         <child link="link_2"/>
-        <axis xyz="0 0 1"/>
-        <limit effort="10" lower="${-0.52}" upper="${pi/2}" velocity="1"/>
+        <axis xyz="0 1 0"/>
         <dynamics damping="0.7"/>
+        <limit effort="100" lower="${-0.52}" upper="${pi/2}" velocity="1"/>
     </joint>
     <!-- *****LINK 3***** -->
@@ -127,4 +143,11 @@
             </material>
         </visual>
+        <xacro:sphere_inertial mass="0.1" radius="${link_2_radius}" o_xyz="0 0 0" o_rpy="0 0 0"/>
+        <collision>
+            <origin xyz="0 0 0" rpy="0 0 0"/>
+            <geometry>
+                <sphere radius="${link_2_radius}"/>
+            </geometry>
+        </collision>
     </link>
     <joint name="1_to_3p" type="fixed">
@@ -135,5 +158,5 @@
     <link name="link_3">
         <visual>
-            <origin xyz="${link_3_length/2} 0 0" rpy="0 ${pi/2} 0"/>
+            <origin xyz="0 0 ${link_3_length/2}" rpy="0 0 0"/>
             <geometry>
                 <cylinder radius="${link_3_radius}" length="${link_3_length}"/>
@@ -143,18 +166,24 @@
             </material>
         </visual>
-        <xacro:cylinder_inertial mass="0.5" radius="${link_3_radius}" length="${link_3_length}" o_xyz="${link_3_length/2} 0 0" o_rpy="0 ${pi/2} 0"/>
+        <xacro:cylinder_inertial mass="1" radius="${link_3_radius}" length="${link_3_length}" o_xyz="0 0 ${link_3_length/2}" o_rpy="0 0 0"/>
+        <collision>
+            <origin xyz="0 0 ${link_3_length/2}" rpy="0 0 0"/>
+            <geometry>
+                <cylinder radius="${link_3_radius}" length="${link_3_length}"/>
+            </geometry>
+        </collision>
     </link>
     <joint name="2_to_3" type="revolute">
-        <origin xyz="${link_2_length} 0 0"/>
+        <origin xyz="${link_2_length} 0 0" rpy="0 0 0"/>
         <parent link="link_2"/>
         <child link="link_3"/>
-        <axis xyz="0 0 1"/>
+        <axis xyz="1 0 0"/>
         <dynamics damping="0.7"/>
-        <limit effort="10" lower="${-pi/2}" upper="${0}" velocity="1"/>
+        <limit effort="100" lower="${-pi/2}" upper="${0}" velocity="1"/>
     </joint>
     <!-- *****LINK 4***** -->
     <link name="link_4">
         <visual>
-            <origin xyz="${-link_4_length/2} 0 0" rpy="0 ${pi/2} 0"/>
+            <origin xyz="0 0 ${link_4_length/2}" rpy="0 0 0"/>
             <geometry>
                 <cylinder radius="${link_4_radius}" length="${link_4_length}"/>
@@ -164,11 +193,16 @@
             </material>
         </visual>
+        <xacro:cylinder_inertial mass="1" radius="${link_4_radius}" length="${link_4_length}" o_xyz="0 0 ${link_4_length/2}" o_rpy="0 0 0"/>
+        <collision>
+            <origin xyz="0 0 ${link_4_length/2}" rpy="0 0 0"/>
+            <geometry>
+                <cylinder radius="${link_4_radius}" length="${link_4_length}"/>
+            </geometry>
+        </collision>
     </link>
     <joint name="3_to_4" type="fixed">
-        <origin xyz="${link_4_length+link_3_length} 0 0"/>
+        <origin xyz="${link_3_length} 0 0" rpy="0 0 0"/>
         <parent link="link_3"/>
         <child link="link_4"/>
-        <axis xyz="0 0 1"/>
-        <dynamics damping="0.7"/>
     </joint>
 </robot>

Commit message: Update robot_1.xacro

File: robot_1.xacro (robot description, xacro)
@@ -77,5 +77,5 @@
     </link>
     <joint name="base_to_1" type="revolute">
-        <origin xyz="0 0 ${base_length}" rpy="0 0 0"/>
+        <origin xyz="0 0 ${base_length + link_1_length/2}" rpy="0 0 0"/>
         <parent link="base_link"/>
         <child link="link_1"/>
@@ -126,5 +126,5 @@
     </link>
     <joint name="1_to_2" type="revolute">
-        <origin xyz="0 0 ${link_1_length}" rpy="0 0 0"/>
+        <origin xyz="0 0 ${link_1_length + link_2_length/2}" rpy="0 0 0"/>
         <parent link="link_1"/>
         <child link="link_2"/>
@@ -175,5 +175,5 @@
     </link>
     <joint name="2_to_3" type="revolute">
-        <origin xyz="${link_2_length} 0 0" rpy="0 0 0"/>
+        <origin xyz="${link_2_length} 0 ${link_3_length/2}" rpy="0 0 0"/>
         <parent link="link_2"/>
         <child link="link_3"/>
@@ -202,5 +202,5 @@
     </link>
     <joint name="3_to_4" type="fixed">
-        <origin xyz="${link_3_length} 0 0" rpy="0 0 0"/>
+        <origin xyz="${link_3_length} 0 ${link_4_length/2}" rpy="0 0 0"/>
         <parent link="link_3"/>
         <child link="link_4"/>
